File: pcb/leds.kicad_sch (KiCad schematic)
At the start: 24 parts

Commit message: Swap to STC8H1K08 and work on JLCPCB assembly support
Parts:
- D1, D2, D3, D4, D5, D6, D7, D8: LCSC (none) -> C157740
- D10, D11, D12, D13, D14, D15, D16, D9: LCSC (none) -> C192316
- R1, R2: LCSC (none) -> C23182
- R3, R4, R5, R6, R7, R8: LCSC (none) -> C23025
Changed lines of the file:
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@@
+			)
+		)
+		(property "LCSC" "C192316"
+			(at 130.81 146.05 0)
+			(effects
+				(font
+					(size 1.27 1.27)
+				)
+				(hide yes)
 			)
 		)
@@
 			)
 		)
+		(property "LCSC" "C23025"
+			(at 182.88 138.43 0)
+			(effects
+				(font
+					(size 1.27 1.27)
+				)
+				(hide yes)
+			)
+		)
 		(pin "1"
 		)
@@
 			)
 		)
+		(property "LCSC" "C157740 "
+			(at 140.97 99.06 0)
+			(effects
+				(font
+					(size 1.27 1.27)
+				)
+				(hide yes)
+			)
+		)
 		(pin "2"
 		)
@@
 			)
 		)
+		(property "LCSC" "C192316"
+			(at 182.88 146.05 0)
+			(effects
+				(font
+					(size 1.27 1.27)
+				)
+				(hide yes)
+			)
+		)
 		(pin "2"
 		)
@@
 			)
 		)
+		(property "LCSC" "C157740 "
+			(at 148.59 99.06 0)
+			(effects
+				(font
+					(size 1.27 1.27)
+				)
+				(hide yes)
+			)
+		)
 		(pin "2"
 		)
@@
 			)
 		)
+		(property "LCSC" "C23182"
+			(at 101.6 85.09 0)
+			(effects
+				(font
+					(size 1.27 1.27)
+				)
+				(hide yes)
+			)
+		)
 		(pin "1"
 		)
@@
 			)
 		)
+		(property "LCSC" "C23025"
+			(at 90.17 138.43 0)
+			(effects
+				(font
+					(size 1.27 1.27)
+				)
+				(hide yes)
+			)
+		)
 		(pin "1"
 		)
@@
 			)
 		)
+		(property "LCSC" "C23025"
+			(at 101.6 138.43 0)
+			(effects
+				(font
+					(size 1.27 1.27)
+				)
+				(hide yes)
+			)
+		)
 		(pin "1"
 		)
@@
 			)
 		)
+		(property "LCSC" "C157740 "
+			(at 132.08 99.06 0)
+			(effects
+				(font
+					(size 1.27 1.27)
+				)
+				(hide yes)
+			)
+		)
 		(pin "2"
 		)
@@
 			)
 		)
+		(property "LCSC" "C23025"
+			(at 121.92 138.43 0)
+			(effects
+				(font
+					(size 1.27 1.27)
+				)
+				(hide yes)
+			)
+		)
 		(pin "1"
 		)
@@
 			)
 		)
+		(property "LCSC" "C157740 "
+			(at 116.84 99.06 0)
+			(effects
+				(font
+					(size 1.27 1.27)
+				)
+				(hide yes)
+			)
+		)
 		(pin "2"
 		)
@@
 			)
 		)
+		(property "LCSC" "C192316"
+			(at 121.92 146.05 0)
+			(effects
+				(font
+					(size 1.27 1.27)
+				)
+				(hide yes)
+			)
+		)
 		(pin "2"
 		)
@@
 			)
 		)
+		(property "LCSC" "C157740 "
+			(at 101.6 99.06 0)
+			(effects
+				(font
+					(size 1.27 1.27)
+				)
+				(hide yes)
+			)
+		)
 		(pin "2"
 		)
@@
 			)
 		)
+		(property "LCSC" "C192316"
+			(at 170.18 146.05 0)
+			(effects
+				(font
+					(size 1.27 1.27)
+				)
+				(hide yes)
+			)
+		)
 		(pin "2"
 		)
@@
 			)
 		)
+		(property "LCSC" "C23182"
+			(at 140.97 85.09 0)
+			(effects
+				(font
+					(size 1.27 1.27)
+				)
+				(hide yes)
+			)
+		)
 		(pin "1"
 		)
@@
 			)
 		)
+		(property "LCSC" "C192316"
+			(at 193.04 146.05 0)
+			(effects
+				(font
+					(size 1.27 1.27)
+				)
+				(hide yes)
+			)
+		)
 		(pin "2"
 		)
@@
 			)
 		)
+		(property "LCSC" "C23025"
+			(at 161.29 138.43 0)
+			(effects
+				(font
+					(size 1.27 1.27)
+				)
+				(hide yes)
+			)
+		)
 		(pin "1"
 		)
@@
 			)
 		)
+		(property "LCSC" "C192316"
+			(at 101.6 146.05 0)
+			(effects
+				(font
+					(size 1.27 1.27)
+				)
+				(hide yes)
+			)
+		)
 		(pin "2"
 		)
@@
 			)
 		)
+		(property "LCSC" "C157740 "
+			(at 109.22 99.06 0)
+			(effects
+				(font
+					(size 1.27 1.27)
+				)
+				(hide yes)
+			)
+		)
 		(pin "2"
 		)
@@
 			)
 		)
+		(property "LCSC" "C157740 "
+			(at 156.21 99.06 0)
+			(effects
+				(font
+					(size 1.27 1.27)
+				)
+				(hide yes)
+			)
+		)
 		(pin "2"
 		)
@@
 			)
 		)
+		(property "LCSC" "C157740 "
+			(at 92.71 99.06 0)
+			(effects
+				(font
+					(size 1.27 1.27)
+				)
+				(hide yes)
+			)
+		)
 		(pin "2"
 		)
@@
 			)
 		)
+		(property "LCSC" "C192316"
+			(at 90.17 146.05 0)
+			(effects
+				(font
+					(size 1.27 1.27)
+				)
+				(hide yes)
+			)
+		)
 		(pin "2"
 		)
@@
 			)
 		)
+		(property "LCSC" "C192316"
+			(at 161.29 146.05 0)
+			(effects
+				(font
+					(size 1.27 1.27)
+				)
+				(hide yes)
+			)
+		)
 		(pin "2"
 		)
@@
 			(at 130.81 138.43 0)
 			(effects
+				(font
+					(size 1.27 1.27)
+				)
+				(hide yes)
+			)
+		)
+		(property "LCSC" "C23025"
+			(at 130.81 138.43 0)
+			(effects

Commit message: More edits to PCB design
 - Change a couple of parts - voltage regulator - to use LCSC parts
 - Increase width of the nametag PCB
 - redo layout a bit
Parts:
- D10, D11, D12, D13, D14, D9: LCSC C192316 -> C5336656
- D15, D16: LCSC C192316 -> C2846641
- renumbered R7 to R3, R8 to R5, R5 to R6, R3 to R7, R6 to R8

Commit message: Update PCB with new naming of PWM channels
Connections:
- net pwm0 is gone; now on net pwm6: R4.1
- net pwm1: now also R7.1; no longer R5.1
- net pwm2: now also R1.1; no longer R3.1
- net pwm3: now also R3.1; no longer R6.1
- net pwm4: now also R8.1; no longer R7.1
- net pwm5: now also R6.1; no longer R8.1
- net pwm6: no longer R1.1
- new net pwm8: R5.1
Other:
- note added: "Eye/Face Top L"
- note added: "Eye/Face Top R"
- note added: "Face Bot C"
- note added: "Face Bot L"
- note added: "Face Bot R"
- note added: "Face Top C"
- note added: "Light L"
- note added: "Light R"

Commit message: Small changes for manufacturability
Parts:
- D10, D11, D12, D13, D14, D9: LCSC C5336656 -> C779453
Other:
- note added: "Check to make sure the PCB footprint agrees with the diode orientation"
Changed lines of the file:
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@@
 		)
 	)
+	(text "Check to make sure the PCB footprint agrees with the diode orientation"
+		(exclude_from_sim no)
+		(at 118.11 73.914 0)
+		(effects
+			(font
+				(size 1.27 1.27)
+			)
+		)
+	)
 	(text "Eye/Face Top L\n"
 		(exclude_from_sim no)
@@
 			)
 		)
-		(property "Datasheet" ""
+		(property "Datasheet" "Teal Green (505nm) or emerald green (520nm) for face"
 			(at 130.81 146.05 0)
 			(hide yes)
@@
 			)
 		)
-		(property "LCSC" "C5336656"
+		(property "LCSC" "C779453"
 			(at 130.81 146.05 0)
 			(hide yes)
@@
 			)
 		)
-		(property "Datasheet" ""
+		(property "Datasheet" "Orange LED for lightsticks"
 			(at 140.97 99.06 0)
 			(hide yes)
@@
 			)
 		)
-		(property "Datasheet" ""
+		(property "Datasheet" "Cyan (496nm) for eyes"
 			(at 182.88 146.05 0)
 			(hide yes)
@@
 			)
 		)
-		(property "Datasheet" ""
+		(property "Datasheet" "Orange LED for lightsticks"
 			(at 148.59 99.06 0)
 			(hide yes)
@@
 			)
 		)
-		(property "Datasheet" ""
+		(property "Datasheet" "Orange LED for lightsticks"
 			(at 132.08 99.06 0)
 			(hide yes)
@@
 			)
 		)
-		(property "Datasheet" ""
+		(property "Datasheet" "Orange LED for lightsticks"
 			(at 116.84 99.06 0)
 			(hide yes)
@@
 			)
 		)
-		(property "Datasheet" ""
+		(property "Datasheet" "Teal Green (505nm) or emerald green (520nm) for face"
 			(at 121.92 146.05 0)
 			(hide yes)
@@
 			)
 		)
-		(property "LCSC" "C5336656"
+		(property "LCSC" "C779453"
 			(at 121.92 146.05 0)
 			(hide yes)
@@
 			)
 		)
-		(property "Datasheet" ""
+		(property "Datasheet" "Orange LED for lightsticks"
 			(at 101.6 99.06 0)
 			(hide yes)
@@
 			)
 		)
-		(property "Datasheet" ""
+		(property "Datasheet" "Teal Green (505nm) or emerald green (520nm) for face"
 			(at 170.18 146.05 0)
 			(hide yes)
@@
 			)
 		)
-		(property "LCSC" "C5336656"
+		(property "LCSC" "C779453"
 			(at 170.18 146.05 0)
 			(hide yes)
@@
 			)
 		)
-		(property "Datasheet" ""
+		(property "Datasheet" "Teal Green (505nm) or emerald green (520nm) for face"
 			(at 193.04 146.05 0)
 			(hide yes)
@@
 			)
 		)
-		(property "LCSC" "C5336656"
+		(property "LCSC" "C779453"
 			(at 193.04 146.05 0)
 			(hide yes)
@@
 			)
 		)
-		(property "Datasheet" ""
+		(property "Datasheet" "Teal Green (505nm) or emerald green (520nm) for face"
 			(at 101.6 146.05 0)
 			(hide yes)
@@
 			)
 		)
-		(property "LCSC" "C5336656"
+		(property "LCSC" "C779453"
 			(at 101.6 146.05 0)
 			(hide yes)
@@
 			)
 		)
-		(property "Datasheet" ""
+		(property "Datasheet" "Orange LED for lightsticks"
 			(at 109.22 99.06 0)
 			(hide yes)
@@
 			)
 		)
-		(property "Datasheet" ""
+		(property "Datasheet" "Orange LED for lightsticks"
 			(at 156.21 99.06 0)
 			(hide yes)
@@
 			)
 		)
-		(property "Datasheet" ""
+		(property "Datasheet" "Orange LED for lightsticks"
 			(at 92.71 99.06 0)
 			(hide yes)
@@
 			)
 		)
-		(property "Datasheet" ""
+		(property "Datasheet" "Teal Green (505nm) or emerald green (520nm) for face"
 			(at 90.17 146.05 0)
 			(hide yes)
@@
 			)
 		)
-		(property "LCSC" "C5336656"
+		(property "LCSC" "C779453"
 			(at 90.17 146.05 0)
 			(hide yes)
@@
 			)
 		)
-		(property "Datasheet" ""
+		(property "Datasheet" "Cyan (496nm) for eyes"
 			(at 161.29 146.05 0)
 			(hide yes)

Commit message: Try swapping to a qfn part instead of tssop-20
Connections:
- net pwm2: now also R6.1; no longer R1.1
- net pwm3: now also R4.1; no longer R3.1
- net pwm5: now also R3.1; no longer R6.1
- net pwm6: now also R1.1; no longer R4.1
Changed lines of the file:
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@@
 	)
 	(label "pwm6"
-		(at 101.6 128.27 0)
+		(at 101.6 80.01 0)
 		(effects
 			(font
@@
 	)
 	(label "pwm2"
-		(at 101.6 80.01 0)
+		(at 130.81 128.27 0)
 		(effects
 			(font
@@
 	)
 	(label "pwm3"
-		(at 90.17 128.27 0)
+		(at 101.6 128.27 0)
 		(effects
 			(font
@@
 	)
 	(label "pwm5"
-		(at 130.81 128.27 0)
+		(at 90.17 129.54 0)
 		(effects
 			(font

Commit message: Update footprints from LCSC EasyEDA Library
Connections:
- net pwm2: now also R8.1; no longer R6.1
- net pwm4: now also R6.1; no longer R8.1
Changed lines of the file:
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@@
 	)
 	(label "pwm4"
-		(at 182.88 128.27 0)
+		(at 130.81 128.27 0)
 		(effects
 			(font
@@
 	)
 	(label "pwm2"
-		(at 130.81 128.27 0)
+		(at 182.88 128.27 0)
 		(effects
 			(font

Commit message: Submit files to JLCPCB for manufacture
Parts:
- D1, D10, D11, D12, D13, D14, D15, D16, D2, D3, D4, D5, D6, D7, D8, D9: footprint LED_SMD:LED_0603_1608Metric_Pad1.05x0.95mm_HandSolder -> LED_SMD:LED_0603_1608Metric
- R1, R2, R3, R4, R5, R6, R7, R8: footprint Resistor_SMD:R_0603_1608Metric_Pad0.98x0.95mm_HandSolder -> Resistor_SMD:R_0603_1608Metric
Changed lines of the file:
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@@
 			)
 		)
-		(property "Footprint" "LED_SMD:LED_0603_1608Metric_Pad1.05x0.95mm_HandSolder"
+		(property "Footprint" "LED_SMD:LED_0603_1608Metric"
 			(at 130.81 146.05 0)
 			(hide yes)
@@
 			)
 		)
-		(property "Footprint" "Resistor_SMD:R_0603_1608Metric_Pad0.98x0.95mm_HandSolder"
+		(property "Footprint" "Resistor_SMD:R_0603_1608Metric"
 			(at 181.102 138.43 90)
 			(hide yes)
@@
 			)
 		)
-		(property "Footprint" "LED_SMD:LED_0603_1608Metric_Pad1.05x0.95mm_HandSolder"
+		(property "Footprint" "LED_SMD:LED_0603_1608Metric"
 			(at 140.97 99.06 0)
 			(hide yes)
@@
 			)
 		)
-		(property "Footprint" "LED_SMD:LED_0603_1608Metric_Pad1.05x0.95mm_HandSolder"
+		(property "Footprint" "LED_SMD:LED_0603_1608Metric"
 			(at 182.88 146.05 0)
 			(hide yes)
@@
 			)
 		)
-		(property "Footprint" "LED_SMD:LED_0603_1608Metric_Pad1.05x0.95mm_HandSolder"
+		(property "Footprint" "LED_SMD:LED_0603_1608Metric"
 			(at 148.59 99.06 0)
 			(hide yes)
@@
 			)
 		)
-		(property "Footprint" "Resistor_SMD:R_0603_1608Metric_Pad0.98x0.95mm_HandSolder"
+		(property "Footprint" "Resistor_SMD:R_0603_1608Metric"
 			(at 99.822 85.09 90)
 			(hide yes)
@@
 			)
 		)
-		(property "Footprint" "Resistor_SMD:R_0603_1608Metric_Pad0.98x0.95mm_HandSolder"
+		(property "Footprint" "Resistor_SMD:R_0603_1608Metric"
 			(at 88.392 138.43 90)
 			(hide yes)
@@
 			)
 		)
-		(property "Footprint" "Resistor_SMD:R_0603_1608Metric_Pad0.98x0.95mm_HandSolder"
+		(property "Footprint" "Resistor_SMD:R_0603_1608Metric"
 			(at 99.822 138.43 90)
 			(hide yes)
@@
 			)
 		)
-		(property "Footprint" "LED_SMD:LED_0603_1608Metric_Pad1.05x0.95mm_HandSolder"
+		(property "Footprint" "LED_SMD:LED_0603_1608Metric"
 			(at 132.08 99.06 0)
 			(hide yes)
@@
 			)
 		)
-		(property "Footprint" "Resistor_SMD:R_0603_1608Metric_Pad0.98x0.95mm_HandSolder"
+		(property "Footprint" "Resistor_SMD:R_0603_1608Metric"
 			(at 120.142 138.43 90)
 			(hide yes)
@@
 			)
 		)
-		(property "Footprint" "LED_SMD:LED_0603_1608Metric_Pad1.05x0.95mm_HandSolder"
+		(property "Footprint" "LED_SMD:LED_0603_1608Metric"
 			(at 116.84 99.06 0)
 			(hide yes)
@@
 			)
 		)
-		(property "Footprint" "LED_SMD:LED_0603_1608Metric_Pad1.05x0.95mm_HandSolder"
+		(property "Footprint" "LED_SMD:LED_0603_1608Metric"
 			(at 121.92 146.05 0)
 			(hide yes)
@@
 			)
 		)
-		(property "Footprint" "LED_SMD:LED_0603_1608Metric_Pad1.05x0.95mm_HandSolder"
+		(property "Footprint" "LED_SMD:LED_0603_1608Metric"
 			(at 101.6 99.06 0)
 			(hide yes)
@@
 			)
 		)
-		(property "Footprint" "LED_SMD:LED_0603_1608Metric_Pad1.05x0.95mm_HandSolder"
+		(property "Footprint" "LED_SMD:LED_0603_1608Metric"
 			(at 170.18 146.05 0)
 			(hide yes)
@@
 			)
 		)
-		(property "Footprint" "Resistor_SMD:R_0603_1608Metric_Pad0.98x0.95mm_HandSolder"
+		(property "Footprint" "Resistor_SMD:R_0603_1608Metric"
 			(at 139.192 85.09 90)
 			(hide yes)
@@
 			)
 		)
-		(property "Footprint" "LED_SMD:LED_0603_1608Metric_Pad1.05x0.95mm_HandSolder"
+		(property "Footprint" "LED_SMD:LED_0603_1608Metric"
 			(at 193.04 146.05 0)
 			(hide yes)
@@
 			)
 		)
-		(property "Footprint" "Resistor_SMD:R_0603_1608Metric_Pad0.98x0.95mm_HandSolder"
+		(property "Footprint" "Resistor_SMD:R_0603_1608Metric"
 			(at 159.512 138.43 90)
 			(hide yes)
@@
 			)
 		)
-		(property "Footprint" "LED_SMD:LED_0603_1608Metric_Pad1.05x0.95mm_HandSolder"
+		(property "Footprint" "LED_SMD:LED_0603_1608Metric"
 			(at 101.6 146.05 0)
 			(hide yes)
@@
 			)
 		)
-		(property "Footprint" "LED_SMD:LED_0603_1608Metric_Pad1.05x0.95mm_HandSolder"
+		(property "Footprint" "LED_SMD:LED_0603_1608Metric"
 			(at 109.22 99.06 0)
 			(hide yes)
@@
 			)
 		)
-		(property "Footprint" "LED_SMD:LED_0603_1608Metric_Pad1.05x0.95mm_HandSolder"
+		(property "Footprint" "LED_SMD:LED_0603_1608Metric"
 			(at 156.21 99.06 0)
 			(hide yes)
@@
 			)
 		)
-		(property "Footprint" "LED_SMD:LED_0603_1608Metric_Pad1.05x0.95mm_HandSolder"
+		(property "Footprint" "LED_SMD:LED_0603_1608Metric"
 			(at 92.71 99.06 0)
 			(hide yes)
@@
 			)
 		)
-		(property "Footprint" "LED_SMD:LED_0603_1608Metric_Pad1.05x0.95mm_HandSolder"
+		(property "Footprint" "LED_SMD:LED_0603_1608Metric"
 			(at 90.17 146.05 0)
 			(hide yes)
@@
 			)
 		)
-		(property "Footprint" "LED_SMD:LED_0603_1608Metric_Pad1.05x0.95mm_HandSolder"
+		(property "Footprint" "LED_SMD:LED_0603_1608Metric"
 			(at 161.29 146.05 0)
 			(hide yes)
@@
 			)
 		)
-		(property "Footprint" "Resistor_SMD:R_0603_1608Metric_Pad0.98x0.95mm_HandSolder"
+		(property "Footprint" "Resistor_SMD:R_0603_1608Metric"
 			(at 129.032 138.43 90)
 			(hide yes)
